File: hardware/magicFlash64.sch (KiCad schematic (older format))
At the start: 35 parts, among them J1 CONN_01X04, J2 Conn_01x07, J3 CONN_01X03, U1 ROMSOCKET, U2 ATMEGA48-20PU, U3 SST39SF040, Y1 20MHz

Commit message: pcb version 0.2
Parts:
- removed D7, D8, D9: D, Diodes_THT:D_DO-35_SOD27_P2.54mm_Vertical_AnodeUp, symbol D
- removed J1: CONN_01X04, Pin_Headers:Pin_Header_Straight_1x04_Pitch2.54mm, symbol CONN_01X04
- removed JP6, JP7: Jumper_NC_Dual, Pin_Headers:Pin_Header_Straight_1x03_Pitch2.54mm, symbol Jumper_NC_Dual
- added C4: 1.2n, Capacitors_THT:C_Disc_D3.4mm_W2.1mm_P2.50mm, symbol C
- added C5: 220p, Capacitors_THT:C_Disc_D3.4mm_W2.1mm_P2.50mm, symbol C
- added J1: 1x4, Pin_Headers:Pin_Header_Straight_1x04_Pitch2.54mm, symbol Conn_01x04
- added J4: 1x4, Pin_Headers:Pin_Header_Straight_1x04_Pitch2.54mm, symbol CONN_01X04
- added R10, R11: 4.7K, Resistors_THT:R_Axial_DIN0204_L3.6mm_D1.6mm_P2.54mm_Vertical, symbol R
- added R12: 100, Resistors_THT:R_Axial_DIN0204_L3.6mm_D1.6mm_P2.54mm_Vertical, symbol R
- added R13: 270, Resistors_THT:R_Axial_DIN0204_L3.6mm_D1.6mm_P2.54mm_Vertical, symbol R
- J2: value Conn_01x07 -> 1x7
- J3: value CONN_01X03 -> 1x3
- JP1, JP2, JP3, JP5: value Jumper_NC_Dual -> 1x3
- JP4: value Jumper -> 1x2
- R9: value 2k -> 100
- U3: value SST39SF040 -> AM29F040
Connections:
- net GND: now also JP1.1, C4.2, C5.1, J4.1 (P1); no longer R9.1, U1.20 (CE)
- net OE: now also R9.2, U1.22 (OE); no longer JP1.1, U2.17 ((PCINT3/OC2/MOSI)PB3)
- net RESET: now also J1.1 (Pin_1)
- net RESTORE: now also R13.2
- net RW: now also J1.3 (Pin_3), R12.1; no longer U2.14 ((PCINT0/CLKO/ICP1)PB0)
- net SEL_A17: now also U3.30 (A17)
- net SEL_A18: now also U3.1 (A18)
- net VCC: now also J4.2 (P2), R10.1, R11.1
- net at U2.3 ((PCINT17/TXD)PD1): now also J4.4 (P4), R11.2
- net at U3.24 (OE): now also R9.1, U2.17 ((PCINT3/OC2/MOSI)PB3), C4.1; no longer R9.2
- net NET: no longer names the net of U2.2 ((PCINT16/RXD)PD0)
- net NET: now also J4.3 (P3), R10.2
- net OE_A11 renamed GND_A11
- net GND_A11: now also U1.20 (CE); no longer U1.22 (OE)
- net OE_EN renamed GPIO
- net GPIO: now also J1.4 (Pin_4)
- new net: C5.2, R12.2, U2.14 ((PCINT0/CLKO/ICP1)PB0)
- new net: J1.2 (Pin_2), R13.1
Other:
- note added: "1-2 28pin with lo ROM (BASIC)\n2-3 28pin without lo ROM (16k slots)\nset to 1-2 for C64"
- note added: "1-2 28pin\n2-3 24pin"
- note added: "C4 \n1.2n ... 407/425/466\n220p ... 469"
- note added: "set 32k slots (requires JP5 to 2-3)\nleave empty for C64"

Commit message: added pcb v0.3 which uses external clock via c64 dot clock
Parts:
- removed C2, C3: 22p, Capacitors_THT:C_Disc_D3.4mm_W2.1mm_P2.50mm, symbol C
- removed C4: 1.2n, Capacitors_THT:C_Disc_D3.4mm_W2.1mm_P2.50mm, symbol C
- removed C5: 220p, Capacitors_THT:C_Disc_D3.4mm_W2.1mm_P2.50mm, symbol C
- removed J1: 1x4, Pin_Headers:Pin_Header_Straight_1x04_Pitch2.54mm, symbol Conn_01x04
- removed R12, R9: 100, Resistors_THT:R_Axial_DIN0204_L3.6mm_D1.6mm_P2.54mm_Vertical, symbol R
- removed R3, R4: 10k, Resistors_THT:R_Axial_DIN0204_L3.6mm_D1.6mm_P2.54mm_Vertical, symbol R
- removed R5, R6, R7, R8: 10K, Resistors_THT:R_Axial_DIN0204_L3.6mm_D1.6mm_P2.54mm_Vertical, symbol R
- removed Y1: 20MHz, Crystals:Crystal_HC18-U_Vertical, symbol Crystal
- added C2: 100n, Capacitors_THT:C_Disc_D3.4mm_W2.1mm_P2.50mm, symbol magicFlash64-rescue:C
- added J1: 1x5, Pin_Headers:Pin_Header_Straight_1x05_Pitch2.54mm, symbol Connector_Generic:Conn_01x05
- added J5: AVR ISP, Pin_Headers:Pin_Header_Straight_2x03_Pitch2.54mm, symbol magicFlash64-rescue:Conn_02x03_Odd_Even
- added RN1: 10k, Resistors_THT:R_Array_SIP7, symbol magicFlash64-rescue:R_Network06
- added U4: 74LS138, Housings_DIP:DIP-16_W7.62mm_Socket, symbol 74xx:74LS138
- C1: symbol C -> magicFlash64-rescue:C
- D1, D2, D3, D4, D5, D6: symbol D -> magicFlash64-rescue:D
- J2: symbol Conn_01x07 -> magicFlash64-rescue:Conn_01x07
- J3: symbol CONN_01X03 -> magicFlash64-rescue:CONN_01X03
- J4: symbol CONN_01X04 -> magicFlash64-rescue:CONN_01X04
- JP1, JP2, JP3, JP5: symbol Jumper_NC_Dual -> magicFlash64-rescue:Jumper_NC_Dual
- JP4: symbol Jumper -> magicFlash64-rescue:Jumper
- R1, R10, R11, R13, R2: symbol R -> magicFlash64-rescue:R
- U1: symbol 27128 -> magicFlash64-rescue:27128
- U2: symbol ATMEGA48-20PU -> magicFlash64-rescue:ATMEGA48-20PU
- U3: symbol SST39SF040 -> magicFlash64-rescue:SST39SF040
Connections:
- net OE is gone; now on net MOSI: U1.22 (OE)
- net GND: now also C2.2, J5.6 (Pin_6), U4.4 (E1), U4.5 (E2), U4.8 (GND)
- net RESET: now also J1.1 (Pin_1)
- net RW: now also U2.14 ((PCINT0/CLKO/ICP1)PB0), J1.3 (Pin_3), U4.2 (A1)
- net SEL_A14: now also RN1.3 (R2)
- net SEL_A15: now also RN1.4 (R3)
- net SEL_A16: now also RN1.5 (R4)
- net SEL_A17: now also RN1.6 (R5)
- net SEL_A18: now also RN1.7 (R6)
- net VCC: now also C2.1, J5.2 (Pin_2), RN1.1 (common), U4.16 (VCC), U4.6 (E3)
- net WE: now also U4.14 (O1); no longer U2.18 ((PCINT4/MISO)PB4)
- net PHI2: now reaches U2.10 ((PCINT7/XTAL2/TOSC2)PB7)
- net PHI2: now also J1.5 (Pin_5), U4.1 (A0)
- net MOSI: now reaches U2.17 ((PCINT3/OC2/MOSI)PB3), U3.24 (OE)
- net MOSI: now also J5.4 (Pin_4)
- net SCL: now reaches J4.3 (P3), R10.2, U2.2 ((PCINT16/RXD)PD0)
- net SDA: now reaches J4.4 (P4), R11.2, U2.3 ((PCINT17/TXD)PD1)
- net DOT_CLK: now reaches U2.9 ((PCINT6/XTAL1/TOSC1)PB6)
- net DOT_CLK: now also J1.4 (Pin_4)
- net at R13.1: now also J1.2 (Pin_2)
- net GPIO renamed SCK
- net SCK: now also D1.2 (A), J2.2 (Pin_2), JP5.3, U3.28 (A13), J5.3 (Pin_3), RN1.2 (R1)
- removed net SEL_A13: D1.2 (A), J2.2 (Pin_2), JP5.3, U2.1 ((PCINT14/~RESET~)PC6), U3.28 (A13)
- new net MISO: J5.1 (Pin_1), U2.18 ((PCINT4/MISO)PB4), U4.3 (A2)
- new net RST: J5.5 (Pin_5), U2.1 ((PCINT14/~RESET~)PC6)
- no-connect marks 1 -> 8
Other:
- note removed: "C4 \n1.2n ... 407/425/466\n220p ... 469"
- moved on the sheet: C1, J3, J4, JP5, R1, R10, R11, R13, R2, U2
